File: Electronics/RC-Endpoint-Limiter/RC-Endpoint-Limiter.sch (KiCad schematic (older format))
At the start: 12 parts

Commit message: added usb port connections decided on smt crystal for usb operation, they seem robust enough
Parts:
- added R? (x2): 22R, symbol Device:R_Small
Connections:
- wire segments 35 -> 42
Other:
- moved on the sheet: J?
Changed lines of the file:
@@
 EESchema Schematic File Version 4
-EELAYER 29 0
+LIBS:RC-Endpoint-Limiter-cache
+EELAYER 30 0
 EELAYER END
 $Descr A4 11693 8268
@@
 L power:GND #PWR?
 U 1 1 5D47C8B5
-P 3450 3000
-F 0 "#PWR?" H 3450 2750 50  0001 C CNN
-F 1 "GND" H 3455 2827 50  0000 C CNN
-F 2 "" H 3450 3000 50  0001 C CNN
-F 3 "" H 3450 3000 50  0001 C CNN
-	1    3450 3000
+P 3200 2750
+F 0 "#PWR?" H 3200 2500 50  0001 C CNN
+F 1 "GND" H 3205 2577 50  0000 C CNN
+F 2 "" H 3200 2750 50  0001 C CNN
+F 3 "" H 3200 2750 50  0001 C CNN
+	1    3200 2750
 	1    0    0    -1
 $EndComp
@@
 	3650 2850 3450 2850
 Wire Wire Line
-	3450 2850 3450 3000
-Wire Wire Line
 	3650 2650 3450 2650
 Wire Wire Line
 	3450 2650 3450 2850
-Connection ~ 3450 2850
 Wire Wire Line
 	3650 2450 3450 2450
@@
 Wire Wire Line
 	4150 3550 4150 3600
+Wire Wire Line
+	3450 2650 3200 2650
+Wire Wire Line
+	3200 2650 3200 2750
+Wire Wire Line
+	4650 3050 2850 3050
 $Comp
 L Connector:USB_B_Micro J?
 U 1 1 5D4913BF
-P 1500 2850
-F 0 "J?" H 1557 3317 50  0000 C CNN
-F 1 "USB_B_Micro" H 1557 3226 50  0000 C CNN
-F 2 "" H 1650 2800 50  0001 C CNN
-F 3 "~" H 1650 2800 50  0001 C CNN
-	1    1500 2850
-	1    0    0    -1
-$EndComp
+P 2550 3250
+F 0 "J?" H 2607 3717 50  0000 C CNN
+F 1 "USB_B_Micro" H 2607 3626 50  0000 C CNN
+F 2 "" H 2700 3200 50  0001 C CNN
+F 3 "~" H 2700 3200 50  0001 C CNN
+	1    2550 3250
+	1    0    0    -1
+$EndComp
+$Comp
+L power:GND #PWR?
+U 1 1 5D49051B
+P 2550 3800
+F 0 "#PWR?" H 2550 3550 50  0001 C CNN
+F 1 "GND" H 2555 3627 50  0000 C CNN
+F 2 "" H 2550 3800 50  0001 C CNN
+F 3 "" H 2550 3800 50  0001 C CNN
+	1    2550 3800
+	1    0    0    -1
+$EndComp
+Wire Wire Line
+	2550 3650 2550 3800
+$Comp
+L Device:R_Small R?
+U 1 1 5D4916F0
+P 3250 3250
+F 0 "R?" V 3200 3100 50  0000 C CNN
+F 1 "22R" V 3200 3400 50  0000 C CNN
+F 2 "" H 3250 3250 50  0001 C CNN
+F 3 "~" H 3250 3250 50  0001 C CNN
+	1    3250 3250
+	0    1    1    0
+$EndComp
+$Comp
+L Device:R_Small R?
+U 1 1 5D491BDA
+P 3250 3350
+F 0 "R?" V 3200 3200 50  0000 C CNN
+F 1 "22R" V 3200 3500 50  0000 C CNN
+F 2 "" H 3250 3350 50  0001 C CNN
+F 3 "~" H 3250 3350 50  0001 C CNN
+	1    3250 3350
+	0    1    1    0
+$EndComp
+Wire Wire Line
+	2850 3250 3150 3250
+Wire Wire Line
+	2850 3350 3150 3350
+Wire Wire Line
+	3350 3350 4650 3350
+Wire Wire Line
+	4650 3250 3350 3250
 $EndSCHEMATC
